File: Schematics/radio-circuit.kicad_sch (KiCad schematic)
At the start: 36 parts, among them J2 STDC14, J3 0, J4 USB_A, U1 USBLC6-2SC6, U2 LD39015M33R, U3 STM32F042F6Px, U4 Si4705-D60-GM, Y1 SG-3030CM

Commit message: Finished component placement
Parts:
- added C1: 100n, Capacitor_SMD:C_0805_2012Metric, symbol Device:C
- added C13, C15: 33p, Capacitor_SMD:C_0402_1005Metric, symbol Device:C
- added C14: 6p, Capacitor_SMD:C_0402_1005Metric, symbol Device:C
- added FB3: 75@100MHz, Inductor_SMD:L_0402_1005Metric, symbol Device:FerriteBead
- added R1: 1M, Resistor_SMD:R_0805_2012Metric, symbol Device:R
- added R11: 22, Resistor_SMD:R_0402_1005Metric, symbol Device:R
- added R13: 330, Resistor_SMD:R_0402_1005Metric, symbol Device:R
- C10: renamed from C9; value 47n -> 100n; footprint Capacitor_SMD:C_0603_1608Metric -> Capacitor_SMD:C_0402_1005Metric; JLCPCB Part Number C1622 -> C307331
- C11: renamed from C10; footprint Capacitor_SMD:C_0603_1608Metric -> Capacitor_SMD:C_0402_1005Metric; JLCPCB Part Number C21122 -> C1532
- C12: renamed from C11; JLCPCB Part Number C1525 -> C307331
- C8: renamed from C7; footprint Capacitor_SMD:C_0402_1005Metric -> Capacitor_SMD:C_0603_1608Metric; JLCPCB Part Number C52923 -> C15849
- renumbered C12 to C16, C1 to C2, C2 to C3, C3 to C4, C4 to C5, C5 to C6, C6 to C7, C8 to C9, J4 to J1, R9 to R10, R10 to R12, R1 to R2, R2 to R3, R3 to R4, R4 to R5, R5 to R6, R6 to R7, R7 to R8, R8 to R9
Connections:
- net +3.3V: now also R11.2; no longer C10.1, Y1.4 (Vcc)
- net FMI: now also C14.1, FB3.1; no longer C16.2, L1.2
- net GND: now also C1.1, C13.2, C14.2, C15.2, R1.1
- net ~{RD_IRQ}: now also R13.1; no longer U4.18 (GPO2/[~{INT}])
- net SHD: now reaches J1.SH (Shield)
- net SHD: now also C1.2, R1.2
- net GPO1: now reaches U4.19 (GPO1)
- net GPO1: now also C13.1
- net V_{FILT} renamed V_{LDO}
- new net GPO2: C15.1, R13.2, U4.18 (GPO2/[~{INT}])
- new net TUNE: C16.2, FB3.2, L1.2
- new net V_{OSC}: C10.1, R11.1, Y1.4 (Vcc)
- no-connect marks 11 -> 9
Other:
- note added: "Extends the ground plane to the USB shield wire and ensures no ESD flows to PCB ground"
- note added: "Pulling ~{SEN} low ensures predictable I2C address for the Si4705"
- note added: "Pulls V_{IO} low while STM32 starts up"
- note added: "Pulls ~{RST} low while STM32 starts up"
- note added: "Reduces reverse oscillation towards the power rail"
- note added: "The datasheet mentions a 10-100nF by-pass capacitor near the Vcc and GND. The 100nF capacitor together with the 22 ohm resistor form a low-pass filter which reduces power rail oscillation caused by the oscillator."
- note removed: "Ensures ~{RST} is held low while STM32 starts up"
- note removed: "Grounding ~{SEN} selects the I2C address of Si4705"
- note removed: "The datasheet mentions a 10-100nF by-pass capacitor near the Vcc and GND. 47uF was chosen due to PCBA provider."
- moved on the sheet: C10, C11, C12, C16, C3, C6, C9, D1, D2, F1, FB1, FB2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

Commit message: Updated JLCPCB part numbers
Parts:
- C14: JLCPCB Part Number C1575 -> C30274
Changed lines of the file:
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@@
 	(wire
 		(pts
+			(xy 246.38 81.28) (xy 250.19 81.28)
+		)
+		(stroke
+			(width 0)
+			(type default)
+		)
+	)
+	(wire
+		(pts
 			(xy 31.75 171.45) (xy 31.75 168.91)
 		)
@@
 	(wire
 		(pts
-			(xy 246.38 81.28) (xy 251.46 81.28)
-		)
-		(stroke
-			(width 0)
-			(type default)
-		)
-	)
-	(wire
-		(pts
 			(xy 38.1 50.8) (xy 45.72 50.8)
 		)
@@
 			)
 		)
-		(property "JLCPCB Part Number" "C1575"
+		(property "JLCPCB Part Number" "C30274"
 			(at 227.33 64.77 0)
 			(hide yes)

Commit message: Finished traces and layers
Other:
- note added: "v0.4"
- note removed: "v0.3"
Changed lines of the file:
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@@
 		)
 	)
-	(text "v0.3"
+	(text "v0.4"
 		(exclude_from_sim no)
 		(at 268.478 193.294 0)
@@
 	(wire
 		(pts
+			(xy 36.83 168.91) (xy 34.29 168.91)
+		)
+		(stroke
+			(width 0)
+			(type default)
+		)
+	)
+	(wire
+		(pts
 			(xy 26.67 50.8) (xy 38.1 50.8)
 		)
@@
 	(wire
 		(pts
+			(xy 34.29 168.91) (xy 34.29 166.37)
+		)
+		(stroke
+			(width 0)
+			(type default)
+		)
+	)
+	(wire
+		(pts
 			(xy 162.56 71.12) (xy 182.88 71.12)
 		)
@@
 	(wire
 		(pts
-			(xy 34.29 166.37) (xy 34.29 168.91)
-		)
-		(stroke
-			(width 0)
-			(type default)
-		)
-	)
-	(wire
-		(pts
 			(xy 58.42 106.68) (xy 63.5 106.68)
 		)
@@
 		)
 		(stroke
-			(width 0)
-			(type default)
-		)
-	)
-	(wire
-		(pts
-			(xy 34.29 168.91) (xy 36.83 168.91)
-		)
-		(stroke

Commit message: Added 3D model for SG-3030CM
Parts:
- Y1: footprint Oscillator:Oscillator_SMD_SeikoEpson_SG3030CM -> Local:Oscillator_SMD_SeikoEpson_SG3030CM
Changed lines of the file:
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@@
 			)
 		)
-		(property "Footprint" "Oscillator:Oscillator_SMD_SeikoEpson_SG3030CM"
+		(property "Footprint" "Local:Oscillator_SMD_SeikoEpson_SG3030CM"
 			(at 241.3 151.13 0)
 			(hide yes)
